Commit message: feat(docs): add project readme
Also updates RGBD camera to pitch 15 degrees upwards to avoid looking at the ground for most of the semantic mapping and navigation. Updated RViz configs.

File: burger_bringup/urdf/turtlebot3_burger_depth.urdf (robot description, URDF)
Before this commit: robot turtlebot3_burger_cam, 10 links, 9 joints
Joints:
- joint camera_joint: origin xyz=0.040 -0.000 0.110 rpy=0 0 0 -> xyz=0.040 -0.000 0.110 rpy=0 -0.2618 0
